File: Hardware/FidoBark.brd (EAGLE design)
At the start: 100 x 80 mm, 37 parts, among them T1 BPX81, U3 HM-10

Commit message: IMU routing complete
jesus that is a tiny package
*ha*
Parts:
- moved C3 72.3 mm to (19.4, 45.2), turned to 180 degrees
- moved C2 69.9 mm to (21.1, 37.8), turned to 180 degrees
- moved R6 66.8 mm to (24.5, 31.4), turned to 270 degrees
- moved U$4 63.1 mm to (22.9, 41.9), turned to 180 degrees
- moved R5 60.4 mm to (21.8, 31.4), turned to 270 degrees
Connections:
- net SCL: now also U$1.19/A5
- net SDA: now also U$1.18/A4
Routing:
- net 3.3V: track 138.2 -> 174.1 mm
- net GND: track 235.6 -> 253.8 mm
- net SDA: track 0.00 -> 8.62 mm
- net SCL: track 0.00 -> 8.45 mm
- net N$8: track 0.00 -> 2.90 mm
- net N$9: track 0.00 -> 2.16 mm

Commit message: mild cleanup
Routing:
- net N$8: track 2.90 -> 3.43 mm
Other:
- board size 100 x 80 mm -> 59.4 x 80 mm
- board text added: "M1"
- board text added: "M2"
Changed lines of the file:
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@@
 <board>
 <plain>
-<wire x1="0" y1="0" x2="100" y2="0" width="0" layer="20"/>
-<wire x1="100" y1="0" x2="100" y2="80" width="0" layer="20"/>
-<wire x1="100" y1="80" x2="0" y2="80" width="0" layer="20"/>
+<wire x1="0" y1="0" x2="59.36" y2="0" width="0" layer="20"/>
+<wire x1="59.36" y1="0" x2="59.36" y2="80" width="0" layer="20"/>
+<wire x1="59.36" y1="80" x2="0" y2="80" width="0" layer="20"/>
 <wire x1="0" y1="80" x2="0" y2="0" width="0" layer="20"/>
 <hole x="2.54" y="2.54" drill="3.048"/>
+<hole x="55.88" y="2.54" drill="3.048"/>
+<text x="15.875" y="2.032" size="1.016" layer="25" font="vector">M1</text>
+<text x="29.591" y="2.159" size="1.016" layer="25" font="vector">M2</text>
 </plain>
 <attributes>
@@
 <attribute name="PROD_ID" value="DIO-08418" x="15.24" y="43.18" size="1.778" layer="27" display="off"/>
 </element>
-<element name="J1" library="SparkFun-Connectors" package="JST-2-SMD" value="" x="10.16" y="5.08" rot="R180">
+<element name="J1" library="SparkFun-Connectors" package="JST-2-SMD" value="" x="10.16" y="5.08" smashed="yes" rot="R180">
 <attribute name="TOP_POS" value="+" x="10.16" y="5.08" size="1.778" layer="27" rot="R180" display="off"/>
 <attribute name="BTM_NEG" value="-" x="10.16" y="5.08" size="1.778" layer="27" rot="R180" display="off"/>
@@
 <attribute name="BTM_POS" value="+" x="10.16" y="5.08" size="1.778" layer="27" rot="R180" display="off"/>
 <attribute name="TOP_NEG" value="-" x="10.16" y="5.08" size="1.778" layer="27" rot="R180" display="off"/>
-</element>
-<element name="JP1" library="pinhead" package="1X02" value="" x="20.32" y="2.54" rot="R180"/>
-<element name="JP2" library="pinhead" package="1X02" value="" x="26.67" y="2.54" rot="R180"/>
+<attribute name="VALUE" x="11.43" y="5.08" size="0.4064" layer="27" rot="R180"/>
+</element>
+<element name="JP1" library="pinhead" package="1X02" value="" x="20.32" y="2.54" smashed="yes" rot="R180">
+<attribute name="VALUE" x="22.86" y="5.715" size="1.27" layer="27" rot="R180"/>
+</element>
+<element name="JP2" library="pinhead" package="1X02" value="" x="26.67" y="2.54" smashed="yes" rot="R180">
+<attribute name="VALUE" x="29.21" y="5.715" size="1.27" layer="27" rot="R180"/>
+</element>
 <element name="R1" library="rcl" package="R0603" value="220" x="12.7" y="38.1" smashed="yes" rot="R90">
 <attribute name="NAME" x="12.065" y="37.465" size="1.27" layer="25" rot="R90"/>
@@
 <attribute name="NAME" x="17.145" y="37.465" size="1.27" layer="25" rot="R90"/>
 </element>
-<element name="R4" library="rcl" package="R0603" value="10k" x="15.24" y="13.97" rot="R180"/>
+<element name="R4" library="rcl" package="R0603" value="10k" x="15.24" y="13.97" smashed="yes" rot="R180">
+<attribute name="NAME" x="15.875" y="13.335" size="1.27" layer="25" rot="R180"/>
+</element>
 <element name="R5" library="rcl" package="R0603" value="10k" x="21.844" y="31.369" smashed="yes" rot="R270">
 <attribute name="NAME" x="22.479" y="32.004" size="1.27" layer="25" rot="R270"/>
@@
 <attribute name="NAME" x="25.146" y="32.004" size="1.27" layer="25" rot="R270"/>
 </element>
-<element name="R7" library="rcl" package="R0603" value="4.7k" x="8.89" y="13.97" rot="R180"/>
+<element name="R7" library="rcl" package="R0603" value="4.7k" x="8.89" y="13.97" smashed="yes" rot="R180">
+<attribute name="NAME" x="9.525" y="13.335" size="1.27" layer="25" rot="R180"/>
+</element>
 <element name="SP1" library="adafruit" package="PS12" value="SPEAKER/PS12" x="33.02" y="49.53" smashed="yes" rot="R180"/>
 <element name="T1" library="opto-trans-siemens" package="BPX81" value="BPX81" x="29.21" y="38.1" smashed="yes" rot="R180">
@@
 </element>
 <element name="U$1" library="Teensy_3_Series_Board_v1.0" package="TEENSY_3.1+4" value="TEENSY_3.1+4" x="22.86" y="26.67" rot="R90"/>
-<element name="U$2" library="adafruit" package="MICROSD" value="MICROSD" x="31.75" y="2.54" rot="R90"/>
+<element name="U$2" library="adafruit" package="MICROSD" value="MICROSD" x="31.75" y="2.54" smashed="yes" rot="R90"/>
 <element name="U$3" library="SparkFun-PowerIC" package="SSOP24" value="TB6612FNG" x="22.86" y="9.525">
 <attribute name="PROD_ID" value="IC-09363" x="22.86" y="9.525" size="1.778" layer="27" display="off"/>
@@
 </element>
 <element name="U$6" library="SparkFun-AnalogIC" package="SOT23-5" value="OPA344" x="-35.56" y="67.31"/>
-<element name="U3" library="HM-10_BLE" package="HM-10" value="HM-10" x="48.26" y="31.75" rot="R180"/>
+<element name="U3" library="HM-10_BLE" package="HM-10" value="HM-10" x="48.26" y="31.75" smashed="yes" rot="R180">
+<attribute name="VALUE" x="45.26" y="34.75" size="1.27" layer="27"/>
+</element>
 <element name="R8" library="adafruit" package="R0603" value="470" x="38.862" y="37.211" smashed="yes" rot="R180">
 <attribute name="NAME" x="40.005" y="39.243" size="1.27" layer="25" rot="R180"/>
@@
 <wire x1="24.511" y1="32.219" x2="24.511" y2="33.401" width="0.4064" layer="1"/>
 <wire x1="24.511" y1="33.401" x2="25.4" y2="34.29" width="0.4064" layer="1"/>
-<wire x1="24.11" y1="39.935" x2="24.11" y2="35.58" width="0.4064" layer="1"/>
-<wire x1="24.11" y1="35.58" x2="25.4" y2="34.29" width="0.4064" layer="1"/>
+<wire x1="25.4" y1="34.29" x2="24.11" y2="35.58" width="0.254" layer="1"/>
+<wire x1="24.11" y1="35.58" x2="24.11" y2="39.935" width="0.254" layer="1"/>
 </signal>
 <signal name="SCL">
@@
 <wire x1="21.844" y1="32.219" x2="21.844" y2="33.274" width="0.4064" layer="1"/>
 <wire x1="21.844" y1="33.274" x2="22.86" y2="34.29" width="0.4064" layer="1"/>
-<wire x1="23.61" y1="39.935" x2="23.61" y2="35.04" width="0.4064" layer="1"/>
-<wire x1="23.61" y1="35.04" x2="22.86" y2="34.29" width="0.4064" layer="1"/>
+<wire x1="22.86" y1="34.29" x2="23.61" y2="35.04" width="0.254" layer="1"/>
+<wire x1="23.61" y1="35.04" x2="23.61" y2="39.935" width="0.254" layer="1"/>
 </signal>
 <signal name="N$8">
 <contactref element="U$4" pad="10"/>
 <contactref element="C3" pad="1"/>
-<wire x1="20.281" y1="45.212" x2="22.61" y2="44.28" width="0.254" layer="1"/>
-<wire x1="22.61" y1="44.28" x2="22.61" y2="43.885" width="0.254" layer="1"/>
+<wire x1="20.281" y1="45.212" x2="22.225" y2="45.212" width="0.254" layer="1"/>
+<wire x1="22.225" y1="45.212" x2="22.606" y2="44.831" width="0.254" layer="1"/>
+<wire x1="22.606" y1="44.831" x2="22.606" y2="43.889" width="0.254" layer="1"/>
+<wire x1="22.606" y1="43.889" x2="22.61" y2="43.885" width="0.254" layer="1"/>
 </signal>
 <signal name="N$9">

Commit message: fucking finished it
goddamn
Parts:
- moved C15 86.1 mm to (23.4, 49.9)
- moved R15 79.2 mm to (15.4, 47.4)
- moved C14 73.7 mm to (15.2, 53.3)
- moved R14 69.4 mm to (10.2, 26.7), turned to 270 degrees
- moved C13 68.4 mm to (11.8, 46.6), turned to 90 degrees
- moved U$6 57.3 mm to (19.1, 50.0), turned to 180 degrees
- moved U$5 48.3 mm to (6.35, 41.9)
- moved R17 47.2 mm to (23.4, 47.8), turned to 180 degrees
- moved R18 43.4 mm to (15.2, 50.8)
- moved R16 36.7 mm to (19.1, 53.3)
Connections:
- net GND: now also U$5.2; no longer U$5.1
- net N$28: now also U$5.1; no longer U$5.2
Routing:
- net ADC_MIC: track 0.00 -> 43.1 mm, vias 0 -> 1
- net GND: track 253.8 -> 284.2 mm
- net 3.3V: track 174.1 -> 202.2 mm, vias 1 -> 2
- net N$28: track 0.00 -> 25.8 mm
- net N$32: track 0.00 -> 10.5 mm
- net N$30: track 0.00 -> 9.17 mm
- net RX: track 60.8 -> 55.6 mm
- net N$29: track 0.00 -> 2.74 mm
- net MISO: track 27.4 -> 28.5 mm
- net N$11: track 5.72 -> 6.43 mm
Other:
- board size 59.4 x 80 mm -> 58.1 x 57.1 mm
- board text added: "Fido"
