File: Hardware/FidoBark.brd (EAGLE design)
At the start: 58.1 x 57.1 mm, 37 parts, among them T1 BPX81, U3 HM-10

Commit message: cosmetics
Other:
- board size 58.1 x 57.1 mm -> 58.1 x 58.4 mm
- board text added: "Joshua Gruenstein Michael Truell"
Changed lines of the file:
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@@
 <plain>
 <wire x1="0" y1="0" x2="58.09" y2="0" width="0" layer="20"/>
-<wire x1="58.09" y1="0" x2="58.09" y2="57.14" width="0" layer="20"/>
-<wire x1="58.09" y1="57.14" x2="0" y2="57.14" width="0" layer="20"/>
-<wire x1="0" y1="57.14" x2="0" y2="0" width="0" layer="20"/>
+<wire x1="58.09" y1="0" x2="58.09" y2="58.41" width="0" layer="20"/>
+<wire x1="58.09" y1="58.41" x2="0" y2="58.41" width="0" layer="20"/>
+<wire x1="0" y1="58.41" x2="0" y2="0" width="0" layer="20"/>
 <hole x="2.54" y="2.54" drill="3.048"/>
 <hole x="55.88" y="2.54" drill="3.048"/>
 <text x="15.875" y="2.032" size="1.016" layer="25" font="vector">M1</text>
 <text x="29.591" y="2.159" size="1.016" layer="25" font="vector">M2</text>
-<hole x="2.54" y="54.61" drill="3.048"/>
-<hole x="55.88" y="54.61" drill="3.048"/>
-<text x="42.672" y="50.038" size="3.81" layer="25">Fido</text>
+<hole x="2.54" y="55.88" drill="3.048"/>
+<hole x="55.88" y="55.88" drill="3.048"/>
+<text x="39.878" y="52.07" size="5.08" layer="25">Fido</text>
+<text x="42.418" y="48.006" size="1.27" layer="25">Joshua Gruenstein
+Michael Truell</text>
 </plain>
 <attributes>
@@
 </board>
 </drawing>
+<compatibility>
+<note version="6.3" minversion="6.2.2" severity="warning">
+Since Version 6.2.2 text objects can contain more than one line,
+which will not be processed correctly with this version.
+</note>
+</compatibility>
 </eagle>
