File: Hardware/FidoBark.brd (EAGLE design)
At the start: 58.1 x 58.4 mm, 37 parts, among them T1 BPX81, U3 HM-10

Commit message: prep for gerber export
Connections:
- removed net VIN: U$1.VIN
- net V_BATT: now also U$1.VIN
Routing:
- net V_BATT: track 29.2 -> 55.7 mm, vias 2 -> 3
Changed lines of the file:
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@@
 <contactref element="U$1" pad="AREF"/>
-</signal>
-<signal name="VIN">
-<contactref element="U$1" pad="VIN"/>
-</signal>
-<signal name="VUSB">
-<contactref element="U$1" pad="VUSB"/>
 </signal>
 <signal name="3.3V">
@@
 <wire x1="14.395" y1="12.275" x2="14.185" y2="12.065" width="0.4064" layer="1"/>
 <wire x1="14.185" y1="12.065" x2="10.414" y2="12.065" width="0.4064" layer="1"/>
-<wire x1="10.414" y1="12.065" x2="8.89" y2="10.541" width="0.4064" layer="1"/>
 <wire x1="8.89" y1="10.541" x2="8.89" y2="8.89" width="0.4064" layer="1"/>
 <wire x1="8.89" y1="8.89" x2="9" y2="8.78" width="0.4064" layer="1"/>
@@
 <wire x1="16.256" y1="10.29" x2="14.395" y2="12.151" width="0.4064" layer="1"/>
 <wire x1="14.395" y1="12.151" x2="14.395" y2="12.275" width="0.4064" layer="1"/>
+<contactref element="U$1" pad="VIN"/>
+<wire x1="10.414" y1="12.065" x2="8.89" y2="10.541" width="0.4064" layer="1"/>
+<wire x1="8.89" y1="10.541" x2="6.858" y2="10.541" width="0.4064" layer="1"/>
+<via x="6.858" y="10.541" extent="1-16" drill="0.6" shape="square"/>
+<wire x1="6.858" y1="10.541" x2="6.35" y2="11.049" width="0.4064" layer="16"/>
+<wire x1="6.35" y1="11.049" x2="6.35" y2="33.02" width="0.4064" layer="16"/>
+<wire x1="6.35" y1="33.02" x2="5.08" y2="34.29" width="0.4064" layer="16"/>
 </signal>
 <signal name="N$2">
@@
 <wire x1="40.093" y1="45.554" x2="39.663" y2="46.99" width="0.4064" layer="1"/>
 </signal>
+<signal name="VUSB">
+<contactref element="U$1" pad="VUSB"/>
+</signal>
 </signals>
