File: Hardware/FidoBark11.sch (EAGLE design)
At the start: 36 parts, among them T1 BPX81, U1 MB85RC256VPF-G-JNERE2

Commit message: cosmetic upgrades
Parts:
- removed R5, R6: 10k, rcl:R-US_R0603
Connections:
- net 3.3V: no longer R5.2, R6.2
- net SCL: no longer R5.1
- net SDA: no longer R6.1
Changed lines of the file:
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@@
 <part name="U$4" library="invensense" deviceset="MPU-9150" device=".QFN"/>
 <part name="SUPPLY3" library="SparkFun-Aesthetics" deviceset="3.3V" device=""/>
-<part name="R5" library="rcl" deviceset="R-US_" device="R0603" value="10k"/>
-<part name="R6" library="rcl" deviceset="R-US_" device="R0603" value="10k"/>
-<part name="SUPPLY4" library="SparkFun-Aesthetics" deviceset="3.3V" device=""/>
 <part name="GND8" library="supply1" deviceset="GND" device=""/>
 <part name="C2" library="rcl" deviceset="C-EU" device="C0603" value="2.2nF"/>
@@
 <instance part="U$4" gate="G$1" x="48.26" y="101.6"/>
 <instance part="SUPPLY3" gate="G$1" x="35.56" y="114.3"/>
-<instance part="R5" gate="G$1" x="66.04" y="101.6" smashed="yes" rot="R270">
-<attribute name="NAME" x="67.5386" y="105.41" size="1.778" layer="95" rot="R270"/>
-<attribute name="VALUE" x="67.818" y="100.33" size="1.778" layer="96" rot="R270"/>
-</instance>
-<instance part="R6" gate="G$1" x="60.96" y="101.6" smashed="yes" rot="R270">
-<attribute name="NAME" x="62.4586" y="105.41" size="1.778" layer="95" rot="R270"/>
-<attribute name="VALUE" x="62.738" y="100.33" size="1.778" layer="96" rot="R270"/>
-</instance>
-<instance part="SUPPLY4" gate="G$1" x="63.5" y="93.98" smashed="yes" rot="R180">
-<attribute name="VALUE" x="69.596" y="92.964" size="1.778" layer="96" rot="R180"/>
-</instance>
 <instance part="GND8" gate="1" x="60.96" y="81.28"/>
 <instance part="C2" gate="G$1" x="27.94" y="101.6"/>
@@
 </segment>
 <segment>
-<pinref part="R6" gate="G$1" pin="2"/>
-<pinref part="SUPPLY4" gate="G$1" pin="3.3V"/>
-<wire x1="60.96" y1="96.52" x2="63.5" y2="93.98" width="0.1524" layer="91"/>
-<pinref part="R5" gate="G$1" pin="2"/>
-<wire x1="66.04" y1="96.52" x2="63.5" y2="93.98" width="0.1524" layer="91"/>
-<junction x="63.5" y="93.98"/>
-</segment>
-<segment>
 <pinref part="R13" gate="G$1" pin="2"/>
 <pinref part="SUPPLY20" gate="G$1" pin="3.3V"/>
@@
 <segment>
 <pinref part="U$4" gate="G$1" pin="SDA"/>
-<wire x1="58.42" y1="111.76" x2="60.96" y2="111.76" width="0.1524" layer="91"/>
-<pinref part="R6" gate="G$1" pin="1"/>
-<wire x1="60.96" y1="111.76" x2="68.58" y2="111.76" width="0.1524" layer="91"/>
-<wire x1="60.96" y1="106.68" x2="60.96" y2="111.76" width="0.1524" layer="91"/>
-<junction x="60.96" y="111.76"/>
+<wire x1="58.42" y1="111.76" x2="68.58" y2="111.76" width="0.1524" layer="91"/>
 <label x="68.58" y="111.76" size="1.016" layer="95" xref="yes"/>
 </segment>
@@
 <segment>
 <pinref part="U$4" gate="G$1" pin="SCL"/>
-<wire x1="58.42" y1="109.22" x2="66.04" y2="109.22" width="0.1524" layer="91"/>
-<pinref part="R5" gate="G$1" pin="1"/>
-<wire x1="66.04" y1="106.68" x2="66.04" y2="109.22" width="0.1524" layer="91"/>
-<wire x1="66.04" y1="109.22" x2="68.58" y2="109.22" width="0.1524" layer="91"/>
-<junction x="66.04" y="109.22"/>
+<wire x1="58.42" y1="109.22" x2="68.58" y2="109.22" width="0.1524" layer="91"/>
 <label x="68.58" y="109.22" size="1.016" layer="95" xref="yes"/>
 </segment>

Commit message: mems microphone
Parts:
- removed C13: 4.7uF, SparkFun-Passives:CAP0603-CAP
- removed C14: 12pF, SparkFun-Passives:CAP0603-CAP
- removed C15: 1uF, SparkFun-Passives:CAP0603-CAP
- removed R14: 2.2k, adafruit:R-US_R0603
- removed R15, R16, R17: 10k, adafruit:R-US_R0603
- removed R18: 1M, adafruit:R-US_R0603
- removed U$5: MIC9.7MM, SparkFun-Sensors:MIC9.7MM
- removed U$6: OPA344, SparkFun-AnalogIC:OPA344
- added U2: ADMP401, SparkFun:ADMP401
Connections:
- removed net N$28: C13.1, R14.1, U$5.1
- removed net N$29: C13.2, R15.1
- removed net N$30: C14.1, R15.2, R18.1, U$6.-IN
- removed net N$32: C15.1, R16.1, R17.2, U$6.+IN
- net 3.3V: now also U2.VDD; no longer R14.2, R16.2, U$6.V+
- net ADC_MIC: now also U2.OUT; no longer C14.2, R18.2, U$6.OUT
- net GND: now also U2.GND@2, U2.GND@4, U2.GND@6; no longer C15.2, R17.1, U$5.2, U$6.V-

Commit message: added esp8266
Parts:
- added R1: 10k, rcl:R-US_R0603
- added U$2: ESP12, esp8266modules:ESP12
Connections:
- new net N$2: R1.2, U$2.CH_PD
- new net RX: U$1.0/RX1/T, U$2.TX
- new net TX: U$1.1/TX1/T, U$2.RX
- net 3.3V: now also R1.1, U$2.VCC
- net GND: now also U$2.GND
Changed lines of the file:
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@@
 <part name="SUPPLY4" library="SparkFun-Aesthetics" deviceset="3.3V" device=""/>
 <part name="GND6" library="supply1" deviceset="GND" device=""/>
+<part name="U$2" library="esp8266modules" deviceset="ESP12" device=""/>
+<part name="SUPPLY12" library="SparkFun-Aesthetics" deviceset="3.3V" device=""/>
+<part name="GND13" library="supply1" deviceset="GND" device=""/>
+<part name="R1" library="rcl" deviceset="R-US_" device="R0603" value="10k"/>
+<part name="SUPPLY13" library="SparkFun-Aesthetics" deviceset="3.3V" device=""/>
 </parts>
 <sheets>
@@
 <instance part="SUPPLY4" gate="G$1" x="121.92" y="124.46" rot="R90"/>
 <instance part="GND6" gate="1" x="121.92" y="104.14"/>
+<instance part="U$2" gate="G$1" x="40.64" y="55.88"/>
+<instance part="SUPPLY12" gate="G$1" x="20.32" y="45.72" rot="R90"/>
+<instance part="GND13" gate="1" x="58.42" y="40.64"/>
+<instance part="R1" gate="G$1" x="15.24" y="58.42"/>
+<instance part="SUPPLY13" gate="G$1" x="7.62" y="58.42" rot="R90"/>
 </instances>
 <busses>
@@
 <pinref part="SUPPLY4" gate="G$1" pin="3.3V"/>
 <wire x1="127" y1="124.46" x2="121.92" y2="124.46" width="0.1524" layer="91"/>
+</segment>
+<segment>
+<pinref part="SUPPLY12" gate="G$1" pin="3.3V"/>
+<pinref part="U$2" gate="G$1" pin="VCC"/>
+<wire x1="20.32" y1="45.72" x2="22.86" y2="45.72" width="0.1524" layer="91"/>
+</segment>
+<segment>
+<pinref part="R1" gate="G$1" pin="1"/>
+<pinref part="SUPPLY13" gate="G$1" pin="3.3V"/>
+<wire x1="10.16" y1="58.42" x2="7.62" y2="58.42" width="0.1524" layer="91"/>
 </segment>
 </net>
@@
 <junction x="121.92" y="109.22"/>
 </segment>
+<segment>
+<pinref part="U$2" gate="G$1" pin="GND"/>
+<pinref part="GND13" gate="1" pin="GND"/>
+<wire x1="55.88" y1="45.72" x2="58.42" y2="45.72" width="0.1524" layer="91"/>
+<wire x1="58.42" y1="45.72" x2="58.42" y2="43.18" width="0.1524" layer="91"/>
+</segment>
 </net>
 <net name="N$1" class="0">
@@
 </segment>
 </net>
+<net name="RX" class="0">
+<segment>
+<pinref part="U$1" gate="G$1" pin="0/RX1/T"/>
+<wire x1="119.38" y1="233.68" x2="116.84" y2="233.68" width="0.1524" layer="91"/>
+<label x="116.84" y="233.68" size="1.016" layer="95" rot="R180" xref="yes"/>
+</segment>
+<segment>
+<pinref part="U$2" gate="G$1" pin="TX"/>
+<wire x1="55.88" y1="63.5" x2="60.96" y2="63.5" width="0.1524" layer="91"/>
+<label x="60.96" y="63.5" size="1.016" layer="95" xref="yes"/>
+</segment>
+</net>
+<net name="TX" class="0">
+<segment>
+<pinref part="U$1" gate="G$1" pin="1/TX1/T"/>
+<wire x1="119.38" y1="231.14" x2="116.84" y2="231.14" width="0.1524" layer="91"/>
+<label x="116.84" y="231.14" size="1.016" layer="95" rot="R180" xref="yes"/>
+</segment>
+<segment>
+<pinref part="U$2" gate="G$1" pin="RX"/>
+<wire x1="55.88" y1="60.96" x2="60.96" y2="60.96" width="0.1524" layer="91"/>
+<label x="60.96" y="60.96" size="1.016" layer="95" xref="yes"/>
+</segment>
+</net>
+<net name="N$2" class="0">
+<segment>
+<pinref part="R1" gate="G$1" pin="2"/>
+<pinref part="U$2" gate="G$1" pin="CH_PD"/>
+<wire x1="20.32" y1="58.42" x2="22.86" y2="58.42" width="0.1524" layer="91"/>
+</segment>
+</net>

Commit message: pcb review cleaning
Parts:
- U2: value ADMP401 -> SPW2430
Connections:
- new net N$6: U$4.AD0
- net GND: no longer U$4.AD0
Other:
- note added: "Nnet Interface"
- note added: "Outputs"
- note added: "Power"
- note added: "Sensors"
- note removed: "Analog Sensors"
- note removed: "Dual Motor Driver"
- note removed: "IMU"
- moved on the sheet: C1, C2, C3, C4, D2, J1, JP1, JP2, R1, R11, R19, R8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

Commit message: corrections 1
Parts:
- added C5, C6, C7: 0.1uF, resistor:C-EUC0603
- R10, R9: value 10k -> 2k
Connections:
- net ADC_BAT renamed ADC_BTR
- removed net N$6: U$4.AD0
- net 3.3V: now also C5.1, C6.1, C7.1
- net GND: now also C5.2, C6.2, C7.2
