File: Hardware/FidoBark11.brd (EAGLE design)
At the start: 50.5 x 44.4 mm, 30 parts, among them T1 BPX81, U1 MB85RC256VPF-G-JNERE2, U2 SPW2430

Commit message: ground plane
forgot this shit again
Routing:
- net GND: track 199.1 -> 200.3 mm
- added copper zone on layer 1, net GND
- added copper zone on layer 16, net GND
Changed lines of the file:
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@@
 <wire x1="6.0325" y1="15.0935" x2="6.0325" y2="9.2075" width="0.3302" layer="1"/>
 <wire x1="6.0325" y1="9.2075" x2="5.715" y2="8.89" width="0.3302" layer="1"/>
-<wire x1="3.44" y1="7.774" x2="3.175" y2="7.509" width="0.4064" layer="1"/>
-<wire x1="3.175" y1="7.509" x2="3.175" y2="2.54" width="0.4064" layer="1"/>
-<wire x1="3.175" y1="2.54" x2="2.413" y2="1.778" width="0.4064" layer="1"/>
-<wire x1="2.413" y1="1.778" x2="1.27" y2="1.778" width="0.4064" layer="1"/>
-<wire x1="1.27" y1="1.778" x2="0.635" y2="2.413" width="0.4064" layer="1"/>
-<wire x1="0.635" y1="2.413" x2="0.635" y2="5.08" width="0.4064" layer="1"/>
-<wire x1="0.635" y1="5.08" x2="1.143" y2="5.588" width="0.4064" layer="1"/>
-<wire x1="1.143" y1="5.588" x2="1.143" y2="6.262" width="0.4064" layer="1"/>
 <wire x1="6.0325" y1="15.0935" x2="6.0325" y2="16.51" width="0.4064" layer="1"/>
 <wire x1="6.0325" y1="16.51" x2="5.9055" y2="16.637" width="0.4064" layer="1"/>
+<polygon width="0.4064" layer="16" isolate="0.3048">
+<vertex x="-1.27" y="-1.27"/>
+<vertex x="52.07" y="-1.27"/>
+<vertex x="52.07" y="45.72"/>
+<vertex x="-1.27" y="45.72"/>
+</polygon>
+<polygon width="0.4064" layer="1" isolate="0.3048">
+<vertex x="-1.27" y="45.72"/>
+<vertex x="52.07" y="45.72"/>
+<vertex x="52.07" y="-1.27"/>
+<vertex x="-1.27" y="-1.27"/>
+</polygon>
+<wire x1="3.44" y1="7.774" x2="3.200403125" y2="5.9342" width="0.4064" layer="1"/>
+<wire x1="3.200403125" y1="5.9342" x2="3.15468125" y2="1.29031875" width="0.4064" layer="1"/>
+<wire x1="3.15468125" y1="1.29031875" x2="3.1343625" y2="1.27" width="0.4064" layer="1"/>
+<wire x1="3.1343625" y1="1.27" x2="1.27" y2="1.27" width="0.4064" layer="1"/>
+<wire x1="1.27" y1="1.27" x2="0.74168125" y2="1.79831875" width="0.4064" layer="1"/>
+<wire x1="0.74168125" y1="1.79831875" x2="0.74168125" y2="4.9911" width="0.4064" layer="1"/>
+<wire x1="0.74168125" y1="4.9911" x2="1.143" y2="5.39241875" width="0.4064" layer="1"/>
+<wire x1="1.143" y1="5.39241875" x2="1.143" y2="6.262" width="0.4064" layer="1"/>
 </signal>
 <signal name="N$1">
